File: elec/layout/bike_light.kicad_pcb (KiCad board)
At the start: 2 copper layers, 40 x 40 mm, 21 parts

Commit message: update the layout according to schematic
Parts:
- J2: footprint Connector_PinHeader_2.54mm:PinHeader_1x02_P2.54mm_Vertical -> Connector_PinHeader_2.54mm:PinHeader_1x03_P2.54mm_Vertical
- R2: value 0.33R -> 1R
- R6: value 75k -> 41.2k
- renumbered D4 to D1, D5 to D2, D1 to D3, D2 to D4, D3 to D5, U2 to U1, U3 to U2, U1 to U3
Connections:
- net 16 renamed 20
- net 17 renamed 21
- net 29 renamed 35
- net 31 renamed 37
- net 39 renamed 42
- net 40 renamed 43
- net 7 renamed 8
- C2 pad 1: 11 -> 14
- C3 pad 1: 15 -> 19
- D1 pad 1: 11 -> 14
- D1 pad 2: 19 -> 23
- D2 pad 1: 12 -> 15
- D3 pad 2: (no net) -> 6
- D4 pad 2: (no net) -> 9
- D5 pad 1: 9 -> 11
- D5 pad 2: (no net) -> 12
- J1 pad A6: 38 -> 41
- J1 pad A8: 41 -> 44
- J1 pad B6: 38 -> 41
- J1 pad B8: 41 -> 44
- J2 pad 2: 12 -> 15
- L1 pad 2: 19 -> 23
- R1 pad 1: 14 -> 18
- R2 pad 1: 11 -> 14
- R4 pad 1: 12 -> 15
- R5 pad 1: 11 -> 14
- U1 pad 1: 12 -> 15
- U1 pad 2: 9 -> 11
- U1 pad 4: 9 -> 11
- U2 pad 1: 12 -> 15
- U3 pad 10: 18 -> 22
- U3 pad 13: 11 -> 14
- U3 pad 18: 19 -> 23
- U3 pad 4: 14 -> 18
- U3 pad 6: 15 -> 19
- U3 pad 9: 18 -> 22
Routing:
- net 12: track 60.7 -> 0.00 mm
- net 15: track 2.25 -> 62.4 mm, vias 0 -> 2
- net 14: track 3.92 -> 29.5 mm, vias 0 -> 2
- net 9: track 18.6 -> 0.00 mm
- net 11: track 29.5 -> 18.6 mm, vias 2 -> 0
- net 1: track 42.6 -> 51.9 mm
- net 23: track 0.00 -> 5.93 mm
- net 19: track 5.93 -> 2.25 mm
- net 18: track 0.50 -> 3.92 mm
- net 22: track 0.00 -> 0.50 mm
